Commit message: corrected some of he nameings and control

File: arm_19/arm_description/robots/robotkolyazilimurdf.urdf (robot description, URDF)
Before this commit: robot arm_description, 8 links, 7 joints
Links:
- removed link 1_eksen_L
- removed link 2_eksen_L
- removed link 3_eksen_L
- removed link 4_eksen_L
- removed link 5_eksen_L
- removed link 6_eksen_L
- added link eksen1_link, mass 1.4155; collision mesh filename=package://arm_description/meshes/1_eksen_L.STL; visual mesh filename=package://arm_description/meshes/1_eksen_L.STL
- added link eksen2_link, mass 1.2949; collision mesh filename=package://arm_description/meshes/2_eksen_L.STL; visual mesh filename=package://arm_description/meshes/2_eksen_L.STL
- added link eksen3_link, mass 2.6432; collision mesh filename=package://arm_description/meshes/3_eksen_L.STL; visual mesh filename=package://arm_description/meshes/3_eksen_L.STL
- added link eksen4_link, mass 1.36543112069823; collision mesh filename=package://arm_description/meshes/4_eksen_L.STL; visual mesh filename=package://arm_description/meshes/4_eksen_L.STL
- added link eksen5_link, mass 2.05411358806035; collision mesh filename=package://arm_description/meshes/5_eksen_L.STL; visual mesh filename=package://arm_description/meshes/5_eksen_L.STL
- added link eksen6_link, mass 0.299295530441066; collision mesh filename=package://arm_description/meshes/6_eksen_L.STL; visual mesh filename=package://arm_description/meshes/6_eksen_L.STL
Joints:
- removed joint 1_eksen_j
- removed joint 2_eksen_j
- removed joint 3_eksen_j
- removed joint 4_eksen_j
- removed joint 5_eksen_j
- removed joint 6_eksen_j
- added joint eksen1_joint: type revolute, parent base_link, child eksen1_link, origin xyz=0.037739 0.0060369 -0.022125 rpy=-1.5708 0 0, axis 0 -1 0, limit lower=-3.14 upper=3.14 effort=10 velocity=20
- added joint eksen2_joint: type revolute, parent eksen1_link, child eksen2_link, origin xyz=0 0.093 0 rpy=-8.6736E-17 8.6736E-17 -1.5708, axis 0 0 -1, limit lower=-1.57 upper=1.57 effort=10 velocity=20
- added joint eksen3_joint: type revolute, parent eksen2_link, child eksen3_link, origin xyz=-0.039 0.41 0 rpy=3.1416 8.6736E-17 -1.5708, axis 0 0 1, limit lower=0 upper=1.57 effort=10 velocity=20
- added joint eksen4_joint: type revolute, parent eksen3_link, child eksen4_link, origin xyz=0.4165 0.065 0.021552 rpy=1.5708 0 1.5708, axis 0 0 -1, limit lower=-3.14 upper=3.14 effort=10 velocity=20
- added joint eksen5_joint: type revolute, parent eksen4_link, child eksen5_link, origin xyz=0.226 -0.007 0.0455 rpy=-1.5708 0 3.1416, axis 0 0 -1, limit lower=-3.14 upper=3.14 effort=10 velocity=20
- added joint eksen6_joint: type revolute, parent eksen5_link, child eksen6_link, origin xyz=0 -0.072 0.088 rpy=1.5708 0.36629 4.0556E-28, axis 0 0 -1, limit lower=-3.14 upper=3.14 effort=10 velocity=20
