Commit message: simplified model again and created a joint robot

File: arm_19/arm_description/robots/arm_description_normal.urdf (robot description, URDF)
Before this commit: robot arm_description, 7 links, 6 joints
Links:
- removed link base_link
- added link arm_base_link, mass 0.22424; collision mesh filename=package://arm_description/meshes/base_link.STL; visual mesh filename=package://arm_description/meshes/base_link.STL
Joints:
- joint joint1: parent base_link -> arm_base_link
