Commit message: Fixed model,move_base and move_group Now all works except sliding

File: arm_19/arm_description/robots/arm_description_with_mobile (copy).urdf (robot description, URDF)
Before this commit: robot arm_description, 13 links, 12 joints
Links:
- removed link anchor
- link base_link: mass None -> 5.00699131277012; geometry collision mesh filename=package://mobile_base_description/meshes/base_link.STL; visual mesh filename=package://mobile_base_description/meshes/base_link.STL
Joints:
- removed joint anchor_joint
- joint joint_dummy: parent anchor -> base_link
- joint left_front_wheel_joint: axis -1 0 0 -> 1 0 0; origin xyz=0.43707 -0.64386 -0.30409 rpy=-1.5708 -2.2837E-18 -3.1043 -> xyz=0.43707 -0.64386 -0.30409 rpy=-1.5708 -2.2837E-18 1.607305; parent anchor -> base_link
- joint left_rear_wheel_joint: axis -1 0 0 -> 1 0 0; origin xyz=0.40294 0.32408 -0.30409 rpy=1.5708 5.545E-15 -3.1043 -> xyz=0.40294 0.32408 -0.30409 rpy=1.5708 5.545E-15 -1.5343; parent anchor -> base_link
- joint right_front_wheel_joint: origin xyz=-0.39172 -0.62476 -0.30409 rpy=0 2.2837E-18 0.037305 -> xyz=-0.34172 -0.43476 -0.30409 rpy=1.5708 2.2837E-18 1.607305; parent anchor -> base_link
- joint right_rear_wheel_joint: origin xyz=-0.42784 0.34311 -0.30409 rpy=0 2.2837E-18 0.037305 -> xyz=-0.42784 0.34311 -0.30409 rpy=1.5708 2.2837E-18 -1.5343; parent anchor -> base_link
