Commit message: fix

File: arm_19/arm_description/robots/arm_description_with_mobile.urdf (robot description, URDF)
Before this commit: robot arm_description, 13 links, 12 joints
Joints:
- joint joint2: limit lower=-3.14 upper=3.14 effort=100 velocity=20 -> lower=-0.70 upper=2.30 effort=100 velocity=20
