Commit message: changed arm and many more

File: arm_19/arm_description/robots/arm_description.urdf (robot description, URDF)
Before this commit: robot arm_description, 8 links, 7 joints
Links:
- removed link eksen1_link
- removed link eksen2_link
- removed link eksen3_link
- removed link eksen4_link
- removed link eksen5_link
- removed link eksen6_link
- added link link1, mass 0.182986637355482; collision mesh filename=package://arm_description/meshes/link1.STL; visual mesh filename=package://arm_description/meshes/link1.STL
- added link link2, mass 0.15891412192705; collision mesh filename=package://arm_description/meshes/link2.STL; visual mesh filename=package://arm_description/meshes/link2.STL
- added link link3, mass 0.12508309667554; collision mesh filename=package://arm_description/meshes/link3.STL; visual mesh filename=package://arm_description/meshes/link3.STL
- added link link4, mass 0.156151945009422; collision mesh filename=package://arm_description/meshes/link4.STL; visual mesh filename=package://arm_description/meshes/link4.STL
- added link link5, mass 0.153675066385186; collision mesh filename=package://arm_description/meshes/link5.STL; visual mesh filename=package://arm_description/meshes/link5.STL
- added link link6, mass 0.299295530441066; collision mesh filename=package://arm_description/meshes/link6.STL; visual mesh filename=package://arm_description/meshes/link6.STL
- link base_link: mass 0.8797 -> 0.22424
Joints:
- removed joint eksen1_joint
- removed joint eksen2_joint
- removed joint eksen3_joint
- removed joint eksen4_joint
- removed joint eksen5_joint
- removed joint eksen6_joint
- removed joint grouding
- added joint joint1: type revolute, parent base_link, child link1, origin xyz=0.055 0.105 0.058 rpy=-1.5708 -6.123E-17 -1.5708, axis 0 1 0, limit lower=-3.14 upper=3.14 effort=100 velocity=20
- added joint joint2: type revolute, parent link1, child link2, origin xyz=0 -0.0975 0.0005 rpy=0.79351 1.5708 0, axis 1 0 0, limit lower=-3.14 upper=3.14 effort=100 velocity=20
- added joint joint3: type revolute, parent link2, child link3, origin xyz=0.0245 0.0495 0.5419 rpy=0.83549 0 3.1416, axis 1 0 0, limit lower=-3.14 upper=3.14 effort=100 velocity=20
- added joint joint4: type revolute, parent link3, child link4, origin xyz=0.0545 0.0355 0.503 rpy=1.5708 -6.9389E-18 1.5708, axis 0 0 1, limit lower=-3.14 upper=3.14 effort=100 velocity=20
- added joint joint5: type revolute, parent link4, child link5, origin xyz=-0.07 0.035 0.044 rpy=1.5708 0 -1.5708, axis 0 0 1, limit lower=-3.14 upper=3.14 effort=100 velocity=20
- added joint joint6: type revolute, parent link5, child link6, origin xyz=-0.041 0.031 0.045 rpy=-1.5708 0 1.5708, axis 0 0 1, limit lower=-3.14 upper=3.14 effort=100 velocity=20
- added joint joint_dummy: type fixed, parent world, child base_link, origin xyz=0 0 0 rpy=0 0 0

Commit message: urdf corrected

File: arm_19/arm_description/robots/arm_description.urdf (robot description, URDF)
Before this commit: robot arm_description, 8 links, 7 joints
Joints:
- joint joint3: axis 1 0 0 -> 0 1 0; origin xyz=0.0245 0.0495 0.5419 rpy=0.83549 0 3.1416 -> xyz=0.0245 0.0495 0.5419 rpy=0 -0.83549 -1.57

File: arm_19/arm_description/robots/arm_description_with_mobile.urdf (robot description, URDF)
Before this commit: robot arm_description, 13 links, 12 joints
Joints:
- joint joint3: axis 1 0 0 -> 0 1 0; origin xyz=0.0245 0.0495 0.5419 rpy=0.83549 0 3.1416 -> xyz=0.0245 0.0495 0.5419 rpy=0 -0.83549 -1.57

Commit message: added camera to the models

File: arm_19/arm_description/robots/arm_description.urdf (robot description, URDF)
Before this commit: robot arm_description, 8 links, 7 joints
Links:
- removed link base_link
- added link arm_base_link, mass 0.22424; collision mesh filename=package://arm_description/meshes/base_link.STL; visual mesh filename=package://arm_description/meshes/base_link.STL
- added link camera_link, mass 1e-5; collision box size=0.05 0.05 0.05; visual box size=0.05 0.05 0.05
Joints:
- added joint camera_joint: type fixed, parent link5, child camera_link, origin xyz=0 0.2 0 rpy=1.57 0 3.14, axis 0 1 0
- joint joint1: parent base_link -> arm_base_link
- joint joint_dummy: child base_link -> arm_base_link

File: arm_19/arm_description/robots/arm_description_with_mobile.urdf (robot description, URDF)
Before this commit: robot arm_description, 13 links, 12 joints
Links:
- added link camera_link, mass 1e-5; collision box size=0.05 0.05 0.05; visual box size=0.05 0.05 0.05
Joints:
- added joint camera_joint: type fixed, parent link5, child camera_link, origin xyz=0 0.2 0 rpy=1.57 0 3.14, axis 0 1 0
